File: Hardware/PortaPAL/PortaPAL.kicad_sch (KiCad schematic)
At the start: 15 parts, among them J1 LCD Display, J2 USB_C_Receptacle_PowerOnly_6P, SW1 SW_Push, SW2 SW_Push, SW3 SW_Push, U1 XC6206PxxxMR

Commit message: added comments and mcu
Parts:
- added J3: JTAG, symbol Connector_Generic:Conn_01x08
- added U2: MSP430FR2422, Package_SO:TSSOP-16_4.4x5mm_P0.65mm, symbol lib:MSP430FR2422
- R1, R2, R3: value R_Small -> 100k
Other:
- note added: "Pin Usage: Package 16 Pins: Fixed: - Power -> 2 pins - Test/NC -> 2 pins - ~{RST} -> 1 pin Remaining 11 pins: - LCD -> 5 pins - Buttons -> 3 pins - IR data -> 2 pins - Battery -> 1 pins Remaining 0 pins"
- note added: "Pins for JTAG: - Vcc - GND - ~{RST} - TEST - TDO - TDI - TMS - TCK"
- note added: "Power Analysis: - Display: Max 300uA - Regulator: Max 1uA - Buttons: Max 3.3uA each - Microcontroller: Max ??? - Charger: Max ???? -> Total: 500uA Battery Capacity: 70mAh Assuming Linear Regulator -> cst current load Total Hours = Capacity / (Total Current) = 70mAh / 0.5mA = 140 hours = 5.8 days at full blast"
- note added: "TODO: - IR communication ? - Maybe only works if charging? - Maybe uart over usb? But then need OTG - Find Suitable microcontroller - Find suitable charging circuit - Programming Connector"
- note removed: "Power Analysis: - Display: Max 300uA - Regulator: Max 1uA - Buttons: Max ??? - Microcontroller: Max ??? - Charger: Max ???? -> Total: 500uA Battery Capacity: 70mAh Assuming Linear Regulator -> cst current load Total Hours = Capacity / (Total Current) = 70mAh / 0.5mA = 140 hours = 5.8 days at full blast"
- note removed: "TODO: - IR communication ? - Maybe only works if charging? - Maybe uart over usb? But then need OTG - Find Suitable microcontroller - Find suitable charging circuit"
Changed lines of the file:
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@@
 		)
 	)
-	(text "TODO:\n\n- IR communication ?\n	- Maybe only works if charging?\n	- Maybe uart over usb? But then need OTG\n- Find Suitable microcontroller\n- Find suitable charging circuit"
-		(exclude_from_sim no)
-		(at 120.396 121.666 0)
+	(text "Pins for JTAG:\n\n- Vcc\n- GND\n- ~{RST}\n- TEST\n\n- TDO\n- TDI\n- TMS\n- TCK"
+		(exclude_from_sim no)
+		(at 63.754 138.43 0)
 		(effects
 			(font
@@
 		)
 	)
-	(text "Power Analysis:\n\n- Display:			Max 300uA\n- Regulator:		Max 1uA\n- Buttons:			Max ???\n- Microcontroller: 	Max ???\n- Charger: 			Max ????\n\n-> Total:			500uA\n\nBattery Capacity: 70mAh\nAssuming Linear Regulator -> cst current load\n\nTotal Hours = Capacity / (Total Current)\n			= 70mAh / 0.5mA = 140 hours = 5.8 days at full blast\n"
+	(text "TODO:\n\n- IR communication ?\n	- Maybe only works if charging?\n	- Maybe uart over usb? But then need OTG\n- Find Suitable microcontroller\n- Find suitable charging circuit\n- Programming Connector"
+		(exclude_from_sim no)
+		(at 121.158 132.842 0)
+		(effects
+			(font
+				(size 1.27 1.27)
+			)
+			(justify left)
+		)
+	)
+	(text "Pin Usage:\n\nPackage 16 Pins:\nFixed:\n- Power 	-> 2 pins\n- Test/NC	-> 2 pins\n- ~{RST}	-> 1 pin\n\nRemaining 11 pins:\n\n- LCD		-> 5 pins\n- Buttons	-> 3 pins\n- IR data	-> 2 pins\n- Battery	-> 1 pins\n\nRemaining 0 pins"
+		(exclude_from_sim no)
+		(at 177.292 69.596 0)
+		(effects
+			(font
+				(size 1.27 1.27)
+			)
+			(justify left)
+		)
+	)
+	(text "Power Analysis:\n\n- Display:			Max 300uA\n- Regulator:		Max 1uA\n- Buttons:			Max 3.3uA each\n- Microcontroller: 	Max ???\n- Charger: 			Max ????\n\n-> Total:			500uA\n\nBattery Capacity: 70mAh\nAssuming Linear Regulator -> cst current load\n\nTotal Hours = Capacity / (Total Current)\n			= 70mAh / 0.5mA = 140 hours = 5.8 days at full blast\n"
 		(exclude_from_sim no)
 		(at 47.752 183.642 0)
@@
 	)
 	(symbol
+		(lib_id "lib:MSP430FR2422")
+		(at 151.13 73.66 0)
+		(unit 1)
+		(exclude_from_sim no)
+		(in_bom yes)
+		(on_board yes)
+		(dnp no)
+		(fields_autoplaced yes)
+		(property "Reference" "U2"
+			(at 151.13 58.42 0)
+			(effects
+				(font
+					(size 1.27 1.27)
+				)
+			)
+		)
+		(property "Value" "MSP430FR2422"
+			(at 151.13 60.96 0)
+			(effects
+				(font
+					(size 1.27 1.27)
+				)
+			)
+		)
+		(property "Footprint" "Package_SO:TSSOP-16_4.4x5mm_P0.65mm"
+			(at 151.13 88.138 0)
+			(effects
+				(font
+					(size 1.27 1.27)
+				)
+				(hide yes)
+			)
+		)
+		(property "Datasheet" "https://www.ti.com/lit/ds/symlink/msp430fr2422.pdf?HQS=dis-dk-null-digikeymode-dsf-pf-null-wwe&ts=1748570568454&ref_url=https%253A%252F%252Fwww.ti.com%252Fgeneral%252Fdocs%252Fsuppproductinfo.tsp%253FdistId%253D10%2526gotoUrl%253Dhttps%253A%252F%252Fwww.ti.com%252Flit%252Fgpn%252Fmsp430fr2422"
+			(at 151.892 80.264 0)
+			(effects
+				(font
+					(size 1.27 1.27)
+				)
+				(hide yes)
+			)
+		)
+		(property "Description" ""
+			(at 151.13 73.66 0)
+			(effects
+				(font
+					(size 1.27 1.27)
+				)
+				(hide yes)
+			)
+		)
+		(pin "13"
+		)
+		(pin "1"
+		)
+		(pin "7"
+		)
+		(pin "6"
+		)
+		(pin "4"
+		)
+		(pin "5"
+		)
+		(pin "16"
+		)
+		(pin "14"
+		)
+		(pin "15"
+		)
+		(pin "8"
+		)
+		(pin "2"
+		)
+		(pin "12"
+		)
+		(pin "3"
+		)
+		(pin "10"
+		)
+		(pin "9"
+		)
+		(pin "11"
+		)
+		(instances
+			(project "PortaPAL"
+				(path "/b2dff3a9-fcd3-4311-bfe3-507200c617d0"
+					(reference "U2")
+					(unit 1)
+				)
+			)
+		)
+	)
+	(symbol
 		(lib_id "Regulator_Linear:XC6206PxxxMR")
 		(at 81.28 33.02 0)
@@
 			)
 		)
-		(property "Value" "R_Small"
+		(property "Value" "100k"
 			(at 224.79 106.6799 0)
 			(effects
@@
 			)
 		)
-		(property "Value" "R_Small"
+		(property "Value" "100k"
 			(at 224.79 132.0799 0)
 			(effects
@@
 	)
 	(symbol
+		(lib_id "Connector_Generic:Conn_01x08")
+		(at 36.83 139.7 0)
+		(mirror y)
+		(unit 1)
+		(exclude_from_sim no)
+		(in_bom yes)
+		(on_board yes)
+		(dnp no)
+		(fields_autoplaced yes)
+		(property "Reference" "J3"
+			(at 36.83 125.73 0)
+			(effects
+				(font
+					(size 1.27 1.27)
+				)
+			)
+		)
+		(property "Value" "JTAG"
+			(at 36.83 128.27 0)
+			(effects
+				(font
+					(size 1.27 1.27)
+				)
+			)
+		)
+		(property "Footprint" ""
+			(at 36.83 139.7 0)
+			(effects
+				(font
+					(size 1.27 1.27)
+				)
+				(hide yes)
+			)
+		)
+		(property "Datasheet" "~"
+			(at 36.83 139.7 0)
+			(effects
+				(font
+					(size 1.27 1.27)
+				)
+				(hide yes)
+			)
+		)
+		(property "Description" "Generic connector, single row, 01x08, script generated (kicad-library-utils/schlib/autogen/connector/)"
+			(at 36.83 139.7 0)
+			(effects
+				(font
+					(size 1.27 1.27)
+				)
+				(hide yes)
+			)
+		)
+		(pin "2"
+		)
+		(pin "1"
+		)
+		(pin "3"
+		)
+		(pin "4"
+		)
+		(pin "5"
+		)
+		(pin "6"
+		)
+		(pin "7"
+		)
+		(pin "8"
+		)
+		(instances
+			(project "PortaPAL"
+				(path "/b2dff3a9-fcd3-4311-bfe3-507200c617d0"
+					(reference "J3")
+					(unit 1)
+				)
+			)
+		)
+	)
+	(symbol
 		(lib_id "power:+BATT")
 		(at 25.4 34.29 0)
@@
 			)
 		)
-		(property "Value" "R_Small"
+		(property "Value" "100k"
 			(at 224.79 119.3799 0)
 			(effects
